File: pcb/TurnsCounter/TurnsCounter.kicad_pcb (KiCad board)
At the start: 2 copper layers, 40 x 80 mm, 39 parts, among them J1 Hall Sensors, J2 PS +9V, J3 I2C, J4 AVR-ISP-10 (SPI), SW1 RESET, SW2 UP, SW3 DOWN, SW4 RETURN, SW5 ENTER, U1 LM317_TO-220, U2 ATmega8A-A, U3 MAX7219, Y1 16MHz

Commit message: pcb alpha, xtal deleted
Parts:
- removed C3, C6: 22p, Capacitor_SMD:C_0805_2012Metric_Pad1.18x1.45mm_HandSolder
- removed Y1: 16MHz, Crystal:Crystal_HC18-U_Vertical
- C1, C4, C5, C9: footprint Capacitor_SMD:CP_Elec_6.3x5.2 -> Capacitor_THT:CP_Radial_D5.0mm_P2.50mm
- C10, C2, C7, R10, R11, R2, R3, R4, R5, R6, R7, R8, R9, U2, U3: moved to B.Cu
- C8: value 10uF -> 1u; footprint Capacitor_SMD:CP_Elec_6.3x5.2 -> Capacitor_SMD:C_0805_2012Metric_Pad1.18x1.45mm_HandSolder; moved to B.Cu
- D1: footprint Diode_THT:D_DO-41_SOD81_P10.16mm_Horizontal -> Diode_THT:D_DO-41_SOD81_P5.08mm_Vertical_KathodeUp
- J2: footprint Converter_DCDC:Converter_DCDC_RECOM_R-78HB-0.5L_THT -> Connector_BarrelJack:BarrelJack_Horizontal
- R1: value 10k -> 240; moved to B.Cu
- moved R7 203.0 mm to (308.7, 22.6), turned to -90 degrees
- moved D2 182.8 mm to (304.8, 16.5)
- moved R5 178.4 mm to (304.6, 22.6), turned to -90 degrees
- moved R6 175.7 mm to (306.6, 22.6), turned to -90 degrees
- moved SW4 174.0 mm to (285.4, 15.0)
- moved U3 162.4 mm to (256.5, 46.2), turned to 180 degrees
- moved SW2 156.6 mm to (295.6, 15.0)
- moved D3 156.2 mm to (237.6, 30.1)
- moved SW5 147.1 mm to (305.6, 26.2)
- moved RV2 142.5 mm to (226.1, 31.9)
- moved SW3 142.2 mm to (295.6, 26.2)
- moved C10 108.7 mm to (255.5, 56.9), turned to 180 degrees
- moved C9 108.6 mm to (254.3, 58.9)
- moved R2 107.9 mm to (210.3, 57.4), turned to 180 degrees
- moved J1 93.4 mm to (183.4, 107.7), turned to 180 degrees
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Connections:
- C8 pad 1: Net-(C8-Pad1) -> GND
- C8 pad 2: GND -> Net-(J4-Pad5)
- J4 pad 5: Net-(C8-Pad1) -> Net-(J4-Pad5)
- R2 pad 2: Net-(C8-Pad1) -> Net-(J4-Pad5)
- SW1 pad 2: Net-(C8-Pad1) -> Net-(J4-Pad5)
- U2 pad 18: unconnected-(U2-Pad18) -> +5V
- U2 pad 29: Net-(C8-Pad1) -> Net-(J4-Pad5)
- U2 pad 7: Net-(C3-Pad1) -> unconnected-(U2-Pad7)
- U2 pad 8: Net-(C6-Pad1) -> unconnected-(U2-Pad8)
Routing:
- net GND: track 0.00 -> 53.7 mm, vias 0 -> 2
- net +5V: track 0.00 -> 47.9 mm
- net Net-(C2-Pad1): track 0.00 -> 17.9 mm
- net Net-(J1-Pad2): track 0.00 -> 14.9 mm
- net Net-(J1-Pad3): track 0.00 -> 11.9 mm
- net Net-(J3-Pad2): track 0.00 -> 11.3 mm
- net Net-(C1-Pad1): track 0.00 -> 10.6 mm
- net Net-(J3-Pad3): track 0.00 -> 9.81 mm
Other:
- outline, holes or cut-outs redrawn

Commit message: ...
Parts:
- moved U3 2.85 mm to (258.3, 44.0), turned to 0 degrees
- moved D3 0.76 mm to (238.3, 30.0)
Changed lines of the file:
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@@
   )
   (footprint "Dawu_PCB_Library:ALS318A" (layer "F.Cu")
-    (at 237.556 30.11)
+    (at 238.31 30)
     (property "Sheetfile" "TurnsCounter.kicad_sch")
     (property "Sheetname" "")
@@
   )
   (footprint "Package_SO:SOIC-24W_7.5x15.4mm_P1.27mm" (layer "B.Cu")
-    (at 256.54 46.228 180)
+    (at 258.31 44)
     (descr "SOIC, 24 Pin (JEDEC MS-013AD, https://www.analog.com/media/en/package-pcb-resources/package/pkg_pdf/soic_wide-rw/RW_24.pdf), generated with kicad-footprint-generator ipc_gullwing_generator.py")
     (tags "SOIC SO")
@@
     (fp_line (start 3.75 7.7) (end 3.75 -7.7) (layer "B.Fab") (width 0.1))
     (fp_line (start 3.75 -7.7) (end -3.75 -7.7) (layer "B.Fab") (width 0.1))
-    (pad "1" smd roundrect (at -4.65 6.985 180) (size 2.05 0.6) (layers "B.Cu" "B.Paste" "B.Mask") (roundrect_rratio 0.25)
+    (pad "1" smd roundrect (at -4.65 6.985) (size 2.05 0.6) (layers "B.Cu" "B.Paste" "B.Mask") (roundrect_rratio 0.25)
       (net 30 "Net-(J4-Pad1)") (pinfunction "DIN") (pintype "input"))
-    (pad "2" smd roundrect (at -4.65 5.715 180) (size 2.05 0.6) (layers "B.Cu" "B.Paste" "B.Mask") (roundrect_rratio 0.25)
+    (pad "2" smd roundrect (at -4.65 5.715) (size 2.05 0.6) (layers "B.Cu" "B.Paste" "B.Mask") (roundrect_rratio 0.25)
       (net 10 "Net-(D3-Pad3)") (pinfunction "DIG_0") (pintype "output"))
-    (pad "3" smd roundrect (at -4.65 4.445 180) (size 2.05 0.6) (layers "B.Cu" "B.Paste" "B.Mask") (roundrect_rratio 0.25)
+    (pad "3" smd roundrect (at -4.65 4.445) (size 2.05 0.6) (layers "B.Cu" "B.Paste" "B.Mask") (roundrect_rratio 0.25)
       (net 18 "Net-(D3-Pad11)") (pinfunction "DIG_4") (pintype "output"))
-    (pad "4" smd roundrect (at -4.65 3.175 180) (size 2.05 0.6) (layers "B.Cu" "B.Paste" "B.Mask") (roundrect_rratio 0.25)
+    (pad "4" smd roundrect (at -4.65 3.175) (size 2.05 0.6) (layers "B.Cu" "B.Paste" "B.Mask") (roundrect_rratio 0.25)
       (net 2 "GND") (pinfunction "GND") (pintype "power_in"))
-    (pad "5" smd roundrect (at -4.65 1.905 180) (size 2.05 0.6) (layers "B.Cu" "B.Paste" "B.Mask") (roundrect_rratio 0.25)
+    (pad "5" smd roundrect (at -4.65 1.905) (size 2.05 0.6) (layers "B.Cu" "B.Paste" "B.Mask") (roundrect_rratio 0.25)
       (net 22 "Net-(D3-Pad15)") (pinfunction "DIG_6") (pintype "output"))
-    (pad "6" smd roundrect (at -4.65 0.635 180) (size 2.05 0.6) (layers "B.Cu" "B.Paste" "B.Mask") (roundrect_rratio 0.25)
+    (pad "6" smd roundrect (at -4.65 0.635) (size 2.05 0.6) (layers "B.Cu" "B.Paste" "B.Mask") (roundrect_rratio 0.25)
       (net 14 "Net-(D3-Pad7)") (pinfunction "DIG_2") (pintype "output"))
-    (pad "7" smd roundrect (at -4.65 -0.635 180) (size 2.05 0.6) (layers "B.Cu" "B.Paste" "B.Mask") (roundrect_rratio 0.25)
+    (pad "7" smd roundrect (at -4.65 -0.635) (size 2.05 0.6) (layers "B.Cu" "B.Paste" "B.Mask") (roundrect_rratio 0.25)
       (net 16 "Net-(D3-Pad9)") (pinfunction "DIG_3") (pintype "output"))
-    (pad "8" smd roundrect (at -4.65 -1.905 180) (size 2.05 0.6) (layers "B.Cu" "B.Paste" "B.Mask") (roundrect_rratio 0.25)
+    (pad "8" smd roundrect (at -4.65 -1.905) (size 2.05 0.6) (layers "B.Cu" "B.Paste" "B.Mask") (roundrect_rratio 0.25)
       (net 24 "Net-(D3-Pad17)") (pinfunction "DIG_7") (pintype "output"))
-    (pad "9" smd roundrect (at -4.65 -3.175 180) (size 2.05 0.6) (layers "B.Cu" "B.Paste" "B.Mask") (roundrect_rratio 0.25)
+    (pad "9" smd roundrect (at -4.65 -3.175) (size 2.05 0.6) (layers "B.Cu" "B.Paste" "B.Mask") (roundrect_rratio 0.25)
       (net 2 "GND") (pinfunction "GND") (pintype "passive"))
-    (pad "10" smd roundrect (at -4.65 -4.445 180) (size 2.05 0.6) (layers "B.Cu" "B.Paste" "B.Mask") (roundrect_rratio 0.25)
+    (pad "10" smd roundrect (at -4.65 -4.445) (size 2.05 0.6) (layers "B.Cu" "B.Paste" "B.Mask") (roundrect_rratio 0.25)
       (net 20 "Net-(D3-Pad13)") (pinfunction "DIG_5") (pintype "output"))
-    (pad "11" smd roundrect (at -4.65 -5.715 180) (size 2.05 0.6) (layers "B.Cu" "B.Paste" "B.Mask") (roundrect_rratio 0.25)
+    (pad "11" smd roundrect (at -4.65 -5.715) (size 2.05 0.6) (layers "B.Cu" "B.Paste" "B.Mask") (roundrect_rratio 0.25)
       (net 12 "Net-(D3-Pad5)") (pinfunction "DIG_1") (pintype "output"))
-    (pad "12" smd roundrect (at -4.65 -6.985 180) (size 2.05 0.6) (layers "B.Cu" "B.Paste" "B.Mask") (roundrect_rratio 0.25)
+    (pad "12" smd roundrect (at -4.65 -6.985) (size 2.05 0.6) (layers "B.Cu" "B.Paste" "B.Mask") (roundrect_rratio 0.25)
       (net 34 "Net-(J4-Pad9)") (pinfunction "LOAD") (pintype "input"))
-    (pad "13" smd roundrect (at 4.65 -6.985 180) (size 2.05 0.6) (layers "B.Cu" "B.Paste" "B.Mask") (roundrect_rratio 0.25)
+    (pad "13" smd roundrect (at 4.65 -6.985) (size 2.05 0.6) (layers "B.Cu" "B.Paste" "B.Mask") (roundrect_rratio 0.25)
       (net 33 "Net-(J4-Pad7)") (pinfunction "CLK") (pintype "input"))
-    (pad "14" smd roundrect (at 4.65 -5.715 180) (size 2.05 0.6) (layers "B.Cu" "B.Paste" "B.Mask") (roundrect_rratio 0.25)
+    (pad "14" smd roundrect (at 4.65 -5.715) (size 2.05 0.6) (layers "B.Cu" "B.Paste" "B.Mask") (roundrect_rratio 0.25)
       (net 13 "Net-(D3-Pad6)") (pinfunction "SEG_A") (pintype "output"))
-    (pad "15" smd roundrect (at 4.65 -4.445 180) (size 2.05 0.6) (layers "B.Cu" "B.Paste" "B.Mask") (roundrect_rratio 0.25)
+    (pad "15" smd roundrect (at 4.65 -4.445) (size 2.05 0.6) (layers "B.Cu" "B.Paste" "B.Mask") (roundrect_rratio 0.25)
       (net 23 "Net-(D3-Pad16)") (pinfunction "SEG_F") (pintype "output"))
-    (pad "16" smd roundrect (at 4.65 -3.175 180) (size 2.05 0.6) (layers "B.Cu" "B.Paste" "B.Mask") (roundrect_rratio 0.25)
+    (pad "16" smd roundrect (at 4.65 -3.175) (size 2.05 0.6) (layers "B.Cu" "B.Paste" "B.Mask") (roundrect_rratio 0.25)
       (net 21 "Net-(D3-Pad14)") (pinfunction "SEG_B") (pintype "output"))
-    (pad "17" smd roundrect (at 4.65 -1.905 180) (size 2.05 0.6) (layers "B.Cu" "B.Paste" "B.Mask") (roundrect_rratio 0.25)
+    (pad "17" smd roundrect (at 4.65 -1.905) (size 2.05 0.6) (layers "B.Cu" "B.Paste" "B.Mask") (roundrect_rratio 0.25)
       (net 19 "Net-(D3-Pad12)") (pinfunction "SEG_G") (pintype "output"))
-    (pad "18" smd roundrect (at 4.65 -0.635 180) (size 2.05 0.6) (layers "B.Cu" "B.Paste" "B.Mask") (roundrect_rratio 0.25)
+    (pad "18" smd roundrect (at 4.65 -0.635) (size 2.05 0.6) (layers "B.Cu" "B.Paste" "B.Mask") (roundrect_rratio 0.25)
       (net 42 "Net-(RV2-Pad2)") (pinfunction "ISET") (pintype "input"))
-    (pad "19" smd roundrect (at 4.65 0.635 180) (size 2.05 0.6) (layers "B.Cu" "B.Paste" "B.Mask") (roundrect_rratio 0.25)
+    (pad "19" smd roundrect (at 4.65 0.635) (size 2.05 0.6) (layers "B.Cu" "B.Paste" "B.Mask") (roundrect_rratio 0.25)
       (net 4 "+5V") (pinfunction "V+") (pintype "power_in"))
-    (pad "20" smd roundrect (at 4.65 1.905 180) (size 2.05 0.6) (layers "B.Cu" "B.Paste" "B.Mask") (roundrect_rratio 0.25)
+    (pad "20" smd roundrect (at 4.65 1.905) (size 2.05 0.6) (layers "B.Cu" "B.Paste" "B.Mask") (roundrect_rratio 0.25)
       (net 9 "Net-(D3-Pad2)") (pinfunction "SEG_C") (pintype "output"))
-    (pad "21" smd roundrect (at 4.65 3.175 180) (size 2.05 0.6) (layers "B.Cu" "B.Paste" "B.Mask") (roundrect_rratio 0.25)
+    (pad "21" smd roundrect (at 4.65 3.175) (size 2.05 0.6) (layers "B.Cu" "B.Paste" "B.Mask") (roundrect_rratio 0.25)
       (net 15 "Net-(D3-Pad8)") (pinfunction "SEG_E") (pintype "output"))
-    (pad "22" smd roundrect (at 4.65 4.445 180) (size 2.05 0.6) (layers "B.Cu" "B.Paste" "B.Mask") (roundrect_rratio 0.25)
+    (pad "22" smd roundrect (at 4.65 4.445) (size 2.05 0.6) (layers "B.Cu" "B.Paste" "B.Mask") (roundrect_rratio 0.25)
       (net 11 "Net-(D3-Pad4)") (pinfunction "SEG_DP") (pintype "output"))
-    (pad "23" smd roundrect (at 4.65 5.715 180) (size 2.05 0.6) (layers "B.Cu" "B.Paste" "B.Mask") (roundrect_rratio 0.25)
+    (pad "23" smd roundrect (at 4.65 5.715) (size 2.05 0.6) (layers "B.Cu" "B.Paste" "B.Mask") (roundrect_rratio 0.25)
       (net 17 "Net-(D3-Pad10)") (pinfunction "SEG_D") (pintype "output"))
-    (pad "24" smd roundrect (at 4.65 6.985 180) (size 2.05 0.6) (layers "B.Cu" "B.Paste" "B.Mask") (roundrect_rratio 0.25)
+    (pad "24" smd roundrect (at 4.65 6.985) (size 2.05 0.6) (layers "B.Cu" "B.Paste" "B.Mask") (roundrect_rratio 0.25)
       (net 52 "unconnected-(U3-Pad24)") (pinfunction "DOUT") (pintype "output"))
     (model "${KICAD6_3DMODEL_DIR}/Package_SO.3dshapes/SOIC-24W_7.5x15.4mm_P1.27mm.wrl"
@@
   (gr_line (start 148.31 125) (end 188.31 125) (layer "Edge.Cuts") (width 0.1))
   (gr_arc (start 158.91 58.65) (mid 162.168501 74.99737) (end 148.31 84.259999) (layer "Edge.Cuts") (width 0.1))
-  (gr_arc (start 200.31 109.48) (mid 200.31 109.48) (end 200.31 109.48) (layer "Edge.Cuts") (width 0.1))
   (segment (start 178 119.9575) (end 172.8175 119.9575) (width 0.5) (layer "B.Cu") (net 1))
   (segment (start 172.72 120.055) (end 172.72 115.635) (width 0.5) (layer "B.Cu") (net 1))

Commit message: First PCB
Parts:
- removed C5: 10uF, Capacitor_THT:CP_Radial_D5.0mm_P2.50mm
- added J10: Conn_01x08_Male, Connector_PinSocket_2.54mm:PinSocket_1x08_P2.54mm_Vertical, F.Cu at (183.2, 80.5)
- added J11: Conn_01x16_Male, Connector_PinSocket_2.54mm:PinSocket_1x16_P2.54mm_Vertical, F.Cu at (215.0, 117.4)
- added J5: RGB Led, Connector_PinSocket_2.54mm:PinSocket_1x04_P2.54mm_Vertical, F.Cu at (152.1, 104.0)
- added J6: RGB Led, Connector_PinSocket_2.54mm:PinSocket_1x04_P2.54mm_Vertical, F.Cu at (207.4, 46.9)
- added J7: Conn_01x06_Male, Connector_PinSocket_2.54mm:PinSocket_1x06_P2.54mm_Vertical, F.Cu at (152.1, 120.6)
- added J8: Keys, Connector_PinSocket_2.54mm:PinSocket_1x06_P2.54mm_Vertical, F.Cu at (190.9, 46.9)
- added J9: Conn_01x08_Male, Connector_PinSocket_2.54mm:PinSocket_1x08_P2.54mm_Vertical, F.Cu at (164.2, 60.2)
- SW3: value DOWN -> CENCEL
- SW4: value RETURN -> DOWN
- moved SW2 118.2 mm to (191.4, 70.9), turned to 90 degrees
- moved SW5 111.5 mm to (199.7, 60.9), turned to 90 degrees
- moved SW3 109.7 mm to (191.4, 60.9), turned to 90 degrees
- moved D2 105.3 mm to (207.5, 56.7)
- moved SW4 102.3 mm to (199.7, 70.9), turned to 90 degrees
- moved R5 101.8 mm to (207.4, 52.8), turned to 90 degrees
- moved R6 101.5 mm to (209.7, 52.8), turned to 90 degrees
- moved R7 101.0 mm to (212.3, 52.8), turned to 90 degrees
- moved D3 94.9 mm to (206.1, 119.3), turned to 90 degrees
- moved U3 91.2 mm to (171.2, 71.0), turned to 90 degrees
- moved C10 73.7 mm to (182.6, 67.8)
- moved C9 70.8 mm to (183.8, 65.3), turned to 180 degrees
- moved RV2 59.0 mm to (181.4, 70.4), turned to 90 degrees
- moved R11 52.2 mm to (200.7, 57.5), turned to 0 degrees
- moved R2 51.8 mm to (173.1, 93.5), turned to 90 degrees
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Connections:
- D2 pad 4: GND -> Net-(D2-Pad4)
- R10 pad 2: GND -> Net-(R10-Pad2)
- R11 pad 2: GND -> Net-(R10-Pad2)
- R7 pad 2: Net-(J4-Pad6) -> Net-(R7-Pad2)
- R8 pad 2: GND -> Net-(R10-Pad2)
- R9 pad 2: GND -> Net-(R10-Pad2)
- RV1 pad 2: unconnected-(RV1-Pad2) -> GND
- SW2 pad 2: +5V -> Net-(SW2-Pad2)
- SW3 pad 2: +5V -> Net-(SW2-Pad2)
- SW4 pad 2: +5V -> Net-(SW2-Pad2)
- SW5 pad 2: +5V -> Net-(SW2-Pad2)
- U2 pad 10: Net-(R10-Pad1) -> Net-(U2-Pad10)
- U2 pad 11: Net-(R11-Pad1) -> Net-(U2-Pad11)
- U2 pad 12: Net-(R5-Pad2) -> Net-(U2-Pad12)
- U2 pad 13: Net-(R6-Pad2) -> Net-(U2-Pad13)
- U2 pad 2: Net-(R8-Pad1) -> Net-(U2-Pad2)
- U2 pad 9: Net-(R9-Pad1) -> Net-(U2-Pad9)
- U3 pad 10: Net-(D3-Pad13) -> Net-(U3-Pad10)
- U3 pad 11: Net-(D3-Pad5) -> Net-(U3-Pad11)
- U3 pad 14: Net-(D3-Pad6) -> Net-(U3-Pad14)
- U3 pad 15: Net-(D3-Pad16) -> Net-(U3-Pad15)
- U3 pad 16: Net-(D3-Pad14) -> Net-(J9-Pad3)
- U3 pad 17: Net-(D3-Pad12) -> Net-(U3-Pad17)
- U3 pad 2: Net-(D3-Pad3) -> Net-(U3-Pad2)
- U3 pad 20: Net-(D3-Pad2) -> Net-(U3-Pad20)
- U3 pad 21: Net-(D3-Pad8) -> Net-(U3-Pad21)
- U3 pad 22: Net-(D3-Pad4) -> Net-(U3-Pad22)
- U3 pad 23: Net-(D3-Pad10) -> Net-(U3-Pad23)
- U3 pad 3: Net-(D3-Pad11) -> Net-(U3-Pad3)
- U3 pad 5: Net-(D3-Pad15) -> Net-(U3-Pad5)
- U3 pad 6: Net-(D3-Pad7) -> Net-(U3-Pad6)
- U3 pad 7: Net-(D3-Pad9) -> Net-(U3-Pad7)
- U3 pad 8: Net-(D3-Pad17) -> Net-(U3-Pad8)
Routing:
- net GND: track 53.7 -> 269.6 mm, vias 2 -> 5
- net +5V: track 47.9 -> 207.2 mm
- net Net-(J4-Pad7): track 0.00 -> 89.3 mm, vias 0 -> 2
- net Net-(J4-Pad1): track 0.00 -> 70.5 mm, vias 0 -> 2
- net Net-(SW2-Pad2): track 0.00 -> 63.8 mm, vias 0 -> 3
- net Net-(J4-Pad6): track 0.00 -> 54.8 mm, vias 0 -> 2
- net Net-(C8-Pad2): track 0.00 -> 54.1 mm, vias 0 -> 2
- net Net-(R10-Pad2): track 0.00 -> 47.5 mm
- net Net-(J4-Pad9): track 0.00 -> 44.3 mm, vias 0 -> 3
- net Net-(U2-Pad2): track 0.00 -> 32.1 mm, vias 0 -> 2
- net Net-(R10-Pad1): track 0.00 -> 26.6 mm
- net Net-(R8-Pad1): track 0.00 -> 26.1 mm
- net Net-(RV2-Pad2): track 0.00 -> 22.4 mm
- net Net-(U2-Pad9): track 0.00 -> 21.9 mm
- net Net-(U2-Pad10): track 0.00 -> 20.7 mm
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Other:
- board size 40 x 80 mm -> 69.2 x 80 mm

Commit message: New PCB with copper area
Routing:
- net +5V: track 207.2 -> 212.1 mm
- net Net-(U3-Pad14): track 6.67 -> 8.99 mm
- net Net-(U3-Pad15): track 6.15 -> 7.29 mm
- net Net-(U3-Pad20): track 6.67 -> 7.72 mm
- net Net-(U3-Pad8): track 5.40 -> 6.38 mm
- net Net-(U3-Pad6): track 7.20 -> 6.45 mm
- net Net-(U3-Pad22): track 8.47 -> 7.72 mm
- added copper zone on B.Cu, net GND
- added copper zone on F.Cu, net GND
- added copper zone on B.Cu, net Net-(D2-Pad4)
