File: pcb/TurnsCounter/TurnsCounter.kicad_pcb (KiCad board)
At the start: 2 copper layers, 69.2 x 80 mm, 42 parts, among them J1 Hall Sensors, J10 Conn_01x08_Male, J11 Conn_01x16_Male, J2 PS +9V, J3 I2C, J4 AVR-ISP-10 (SPI), J5 RGB Led, J6 RGB Led, J7 Conn_01x06_Male, J8 Keys, J9 Conn_01x08_Male, SW1 RESET, SW2 UP, SW3 CENCEL, SW4 DOWN, SW5 ENTER, U1 LM317_TO-220, U2 ATmega8A-A, U3 MAX7219

Commit message: Pcb...
Routing:
- net Net-(U2-Pad11): track 20.6 -> 25.0 mm
- net Net-(U2-Pad10): track 20.7 -> 23.3 mm
- net Net-(U2-Pad2): track 32.1 -> 31.1 mm
- net Net-(U2-Pad12): track 20.4 -> 19.5 mm
Changed lines of the file:
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@@
   (segment (start 214.985 55.511) (end 212.321 58.175) (width 0.5) (layer "B.Cu") (net 55))
   (segment (start 214.985 46.895) (end 214.985 55.511) (width 0.5) (layer "B.Cu") (net 55))
+  (segment (start 166.940112 101.924888) (end 165.225958 103.63904) (width 0.5) (layer "B.Cu") (net 56))
+  (segment (start 165.225958 103.63904) (end 162.605204 103.63904) (width 0.5) (layer "B.Cu") (net 56))
+  (segment (start 162.605204 103.63904) (end 159.966653 101.000489) (width 0.5) (layer "B.Cu") (net 56))
   (segment (start 159.966653 101.000489) (end 155.164511 101.000489) (width 0.5) (layer "B.Cu") (net 56))
-  (segment (start 164.185 104.68) (end 163.646164 104.68) (width 0.5) (layer "B.Cu") (net 56))
-  (segment (start 163.646164 104.68) (end 159.966653 101.000489) (width 0.5) (layer "B.Cu") (net 56))
-  (segment (start 166.940112 101.924888) (end 164.185 104.68) (width 0.5) (layer "B.Cu") (net 56))
+  (segment (start 155.164511 101.000489) (end 152.12 104.045) (width 0.5) (layer "B.Cu") (net 56))
   (segment (start 168.5725 101.924888) (end 166.940112 101.924888) (width 0.5) (layer "B.Cu") (net 56))
-  (segment (start 155.164511 101.000489) (end 152.12 104.045) (width 0.5) (layer "B.Cu") (net 56))
   (segment (start 160.261146 100.235) (end 154.870019 100.235) (width 0.5) (layer "B.Cu") (net 57))
   (segment (start 168.5725 101.124888) (end 166.68013 101.124888) (width 0.5) (layer "B.Cu") (net 57))
@@
   (via (at 174.98 108.49) (size 2.5) (drill 0.6) (layers "F.Cu" "B.Cu") (free) (net 59))
   (via (at 167.36 107.855) (size 2.5) (drill 0.6) (layers "F.Cu" "B.Cu") (free) (net 59))
-  (segment (start 159.455978 111.665) (end 159.436489 111.684489) (width 0.5) (layer "B.Cu") (net 59))
-  (segment (start 154.77452 115.36048) (end 152.12 118.015) (width 0.5) (layer "B.Cu") (net 59))
+  (segment (start 159.181456 112.208544) (end 159.181456 113.371456) (width 0.5) (layer "B.Cu") (net 59))
+  (segment (start 162.28 111.665) (end 159.725 111.665) (width 0.5) (layer "B.Cu") (net 59))
+  (segment (start 174.8225 108.3325) (end 174.98 108.49) (width 0.5) (layer "B.Cu") (net 59))
+  (segment (start 174.8225 105.774888) (end 174.8225 108.3325) (width 0.5) (layer "B.Cu") (net 59))
+  (segment (start 159.181456 113.371456) (end 154.537912 118.015) (width 0.5) (layer "B.Cu") (net 59))
   (segment (start 167.36 107.855) (end 166.09 107.855) (width 0.5) (layer "B.Cu") (net 59))
-  (segment (start 174.8225 108.3325) (end 174.98 108.49) (width 0.5) (layer "B.Cu") (net 59))
-  (segment (start 162.28 111.665) (end 161.014944 111.665) (width 0.5) (layer "B.Cu") (net 59))
-  (segment (start 174.8225 105.774888) (end 174.8225 108.3325) (width 0.5) (layer "B.Cu") (net 59))
-  (segment (start 155.509964 111.665) (end 154.77452 112.400444) (width 0.5) (layer "B.Cu") (net 59))
+  (segment (start 159.725 111.665) (end 159.181456 112.208544) (width 0.5) (layer "B.Cu") (net 59))
+  (segment (start 154.537912 118.015) (end 152.12 118.015) (width 0.5) (layer "B.Cu") (net 59))
   (segment (start 166.09 107.855) (end 162.28 111.665) (width 0.5) (layer "B.Cu") (net 59))
-  (segment (start 154.77452 112.400444) (end 154.77452 115.36048) (width 0.5) (layer "B.Cu") (net 59))
-  (segment (start 161.014944 111.665) (end 155.509964 111.665) (width 0.5) (layer "B.Cu") (net 59))
+  (segment (start 152.64452 115.99952) (end 152.12 115.475) (width 0.5) (layer "B.Cu") (net 60))
+  (segment (start 155.651465 115.841465) (end 155.493409 115.99952) (width 0.5) (layer "B.Cu") (net 60))
+  (segment (start 158.431936 113.060994) (end 155.651465 115.841465) (width 0.5) (layer "B.Cu") (net 60))
+  (segment (start 161.75952 110.91548) (end 159.414538 110.91548) (width 0.5) (layer "B.Cu") (net 60))
+  (segment (start 158.431936 111.898083) (end 158.431936 113.060994) (width 0.5) (layer "B.Cu") (net 60))
+  (segment (start 168.350112 104.324888) (end 161.75952 110.91548) (width 0.5) (layer "B.Cu") (net 60))
+  (segment (start 155.493409 115.99952) (end 152.64452 115.99952) (width 0.5) (layer "B.Cu") (net 60))
   (segment (start 168.5725 104.324888) (end 168.350112 104.324888) (width 0.5) (layer "B.Cu") (net 60))
-  (segment (start 154.025 113.57) (end 152.12 115.475) (width 0.5) (layer "B.Cu") (net 60))
-  (segment (start 168.350112 104.324888) (end 161.75952 110.91548) (width 0.5) (layer "B.Cu") (net 60))
-  (segment (start 155.199502 110.91548) (end 154.025 112.089982) (width 0.5) (layer "B.Cu") (net 60))
-  (segment (start 154.025 112.089982) (end 154.025 113.57) (width 0.5) (layer "B.Cu") (net 60))
-  (segment (start 161.75952 110.91548) (end 155.199502 110.91548) (width 0.5) (layer "B.Cu") (net 60))
-  (segment (start 167.474888 103.524888) (end 167.147509 103.852267) (width 0.5) (layer "B.Cu") (net 61))
-  (segment (start 167.147509 103.852267) (end 167.147509 104.467509) (width 0.5) (layer "B.Cu") (net 61))
-  (segment (start 167.147509 104.467509) (end 161.449058 110.16596) (width 0.5) (layer "B.Cu") (net 61))
-  (segment (start 168.5725 103.524888) (end 167.474888 103.524888) (width 0.5) (layer "B.Cu") (net 61))
-  (segment (start 161.449058 110.16596) (end 154.88904 110.16596) (width 0.5) (layer "B.Cu") (net 61))
-  (segment (start 154.88904 110.16596) (end 152.12 112.935) (width 0.5) (layer "B.Cu") (net 61))
+  (segment (start 159.414538 110.91548) (end 158.431936 111.898083) (width 0.5) (layer "B.Cu") (net 60))
+  (segment (start 161.449058 110.16596) (end 167.147509 104.467509) (width 0.5) (layer "B.Cu") (net 61))
+  (segment (start 167.474888 103.524888) (end 168.5725 103.524888) (width 0.5) (layer "B.Cu") (net 61))
+  (segment (start 159.104076 110.165961) (end 161.449058 110.16596) (width 0.5) (layer "B.Cu") (net 61))
+  (segment (start 167.147509 103.852267) (end 167.474888 103.524888) (width 0.5) (layer "B.Cu") (net 61))
+  (segment (start 157.682416 111.587622) (end 159.104076 110.165961) (width 0.5) (layer "B.Cu") (net 61))
+  (segment (start 167.147509 104.467509) (end 167.147509 103.852267) (width 0.5) (layer "B.Cu") (net 61))
+  (segment (start 152.12 112.935) (end 154.435 115.25) (width 0.5) (layer "B.Cu") (net 61))
+  (segment (start 157.682416 112.750532) (end 157.682416 111.587622) (width 0.5) (layer "B.Cu") (net 61))
+  (segment (start 155.182948 115.25) (end 157.682416 112.750532) (width 0.5) (layer "B.Cu") (net 61))
+  (segment (start 154.435 115.25) (end 155.182948 115.25) (width 0.5) (layer "B.Cu") (net 61))
   (segment (start 159.44856 109.41644) (end 160.08356 109.41644) (width 0.5) (layer "B.Cu") (net 62))
-  (segment (start 152.12 110.395) (end 153.09856 109.41644) (width 0.5) (layer "B.Cu") (net 62))
-  (segment (start 153.09856 109.41644) (end 159.44856 109.41644) (width 0.5) (layer "B.Cu") (net 62))
   (segment (start 166.397989 104.157047) (end 161.138596 109.41644) (width 0.5) (layer "B.Cu") (net 62))
+  (segment (start 158.793615 109.416441) (end 156.716483 111.493573) (width 0.5) (layer "B.Cu") (net 62))
   (segment (start 167.214906 102.724888) (end 166.397989 103.541805) (width 0.5) (layer "B.Cu") (net 62))
   (segment (start 161.138596 109.41644) (end 159.44856 109.41644) (width 0.5) (layer "B.Cu") (net 62))
+  (segment (start 155.622966 113.75) (end 153.994982 113.75) (width 0.5) (layer "B.Cu") (net 62))
+  (segment (start 153.56 111.835) (end 152.12 110.395) (width 0.5) (layer "B.Cu") (net 62))
   (segment (start 166.397989 103.541805) (end 166.397989 104.157047) (width 0.5) (layer "B.Cu") (net 62))
+  (segment (start 156.716483 112.656483) (end 155.622966 113.75) (width 0.5) (layer "B.Cu") (net 62))
+  (segment (start 156.716483 111.493573) (end 156.716483 112.656483) (width 0.5) (layer "B.Cu") (net 62))
   (segment (start 167.309888 102.724888) (end 167.214906 102.724888) (width 0.5) (layer "B.Cu") (net 62))
+  (segment (start 159.44856 109.41644) (end 158.793615 109.416441) (width 0.5) (layer "B.Cu") (net 62))
+  (segment (start 153.994982 113.75) (end 153.56 113.315018) (width 0.5) (layer "B.Cu") (net 62))
   (segment (start 168.5725 102.724888) (end 167.309888 102.724888) (width 0.5) (layer "B.Cu") (net 62))
+  (segment (start 153.56 113.315018) (end 153.56 111.835) (width 0.5) (layer "B.Cu") (net 62))
   (segment (start 190.855 50.07) (end 195.935 50.07) (width 0.5) (layer "F.Cu") (net 63))
   (segment (start 195.935 50.07) (end 204.19 50.07) (width 0.5) (layer "F.Cu") (net 63))

Commit message: pdf
Routing:
- added copper zone on F.Cu, net Net-(D2-Pad4)
Changed lines of the file:
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@@
+    )
+  )
+  (zone (net 55) (net_name "Net-(D2-Pad4)") (layer "F.Cu") (hatch edge 0.508)
+    (connect_pads (clearance 0.508))
+    (min_thickness 0.254) (filled_areas_thickness no)
+    (fill yes (thermal_gap 0.508) (thermal_bridge_width 0.508))
+    (polygon
+      (pts
+        (xy 217.525 125)
+        (xy 188.95 125)
+        (xy 188.95 44.99)
+        (xy 217.525 44.99)
+      )
     )
   )

Commit message: pcb fin
Parts:
- SW1, SW2, SW3, SW4, SW5: footprint Button_Switch_THT:SW_PUSH_6mm -> Dawu_PCB_Library:SW_PUSH_6mm_2
Routing:
- net Net-(J9-Pad1): track 8.99 -> 0.00 mm
- net Net-(J4-Pad7): track 89.3 -> 96.0 mm
- net Net-(J10-Pad4): track 6.45 -> 8.14 mm
- net Net-(J8-Pad6): track 47.5 -> 49.1 mm
- net Net-(J10-Pad6): track 6.38 -> 5.40 mm
- net Net-(J10-Pad2): track 7.21 -> 8.11 mm
- net Net-(J8-Pad2): track 26.1 -> 26.9 mm
- net Net-(J4-Pad1): track 70.5 -> 69.9 mm
- net Net-(J9-Pad2): track 7.29 -> 6.71 mm
